File: hardware/TeleprinterHat/TeleprinterHat.kicad_pcb (KiCad board)
At the start: 2 copper layers, 141 parts, among them J1 RJ12, J2 RJ12, J4 USB_B_Micro, J5 RS232, J6 JTAG, J7 RasPi GPIO, K1 EA2-5NU, Q1 STD25NF20, Q10 FMMT625, Q2 MMBT3904, Q3 FMMT625, Q4 FMMT625, Q5 MMBT5551L, Q6 MMBT5551L, Q7 MMBTA42L, Q8 SQ2325ES, Q9 FMMT597, U1 NCP1117-3.3_TO252, U10 TLV3502, U11 MCP6004, U13 74LVC1G04, U14 STM32F103C8Tx, U2 74LVC1G04, U3 FT232RL, U4 MAX3232, U5 MC34063, U6 24LC32AT-IOT, U7 SFH690BT, U8 SFH690BT, U9 IR44273, Y1 8MHz

Commit message: Almost ready!
Parts:
- removed JP10: CURR1, Connector_PinHeader_2.54mm:PinHeader_1x02_P2.54mm_Vertical
- removed JP15: TPBAUD0, Connector_PinHeader_2.54mm:PinHeader_1x02_P2.54mm_Vertical
- removed JP16: TPBAUD1, Connector_PinHeader_2.54mm:PinHeader_1x02_P2.54mm_Vertical
- removed JP2: VOLT0, Connector_PinHeader_2.54mm:PinHeader_1x02_P2.54mm_Vertical
- removed JP20: TEST1, Connector_PinHeader_2.54mm:PinHeader_1x02_P2.54mm_Vertical
- removed JP21: TEST2, Connector_PinHeader_2.54mm:PinHeader_1x02_P2.54mm_Vertical
- removed JP3: VOLT1, Connector_PinHeader_2.54mm:PinHeader_1x02_P2.54mm_Vertical
- removed JP7: HBAUD0, Connector_PinHeader_2.54mm:PinHeader_1x02_P2.54mm_Vertical
- removed JP8: HBAUD1, Connector_PinHeader_2.54mm:PinHeader_1x02_P2.54mm_Vertical
- removed JP9: CURR0, Connector_PinHeader_2.54mm:PinHeader_1x02_P2.54mm_Vertical
- added H1: MountingHole, MountingHole:MountingHole_2.7mm_M2.5, F.Cu at (89.0, 90.0)
- added H2: MountingHole, MountingHole:MountingHole_2.7mm_M2.5, F.Cu at (89.0, 41.0)
- added H3: MountingHole, MountingHole:MountingHole_2.7mm_M2.5, F.Cu at (147.0, 90.0)
- added H4: MountingHole, MountingHole:MountingHole_2.7mm_M2.5, F.Cu at (147.0, 41.0)
- added H5: MountingHole, MountingHole:MountingHole_2.7mm_M2.5, F.Cu at (147.0, 110.0)
- added H6: MountingHole, MountingHole:MountingHole_2.7mm_M2.5, F.Cu at (70.5, 26.5)
- added H7: MountingHole, MountingHole:MountingHole_2.7mm_M2.5, F.Cu at (70.5, 110.0)
- added H8: MountingHole, MountingHole:MountingHole_2.7mm_M2.5, F.Cu at (147.0, 26.5)
- added J10: Conn_01x01_Male, Connector_PinHeader_2.54mm:PinHeader_1x01_P2.54mm_Vertical, F.Cu at (115.9, 81.8)
- added J11: Conn_01x01_Male, Connector_PinHeader_2.54mm:PinHeader_1x01_P2.54mm_Vertical, F.Cu at (102.1, 60.1)
- added J3: DC_JACK, Connector_BarrelJack:BarrelJack_Wuerth_6941xx301002, F.Cu at (92.3, 29.2)
- added J8: Conn_01x01_Male, Connector_PinHeader_2.54mm:PinHeader_1x01_P2.54mm_Vertical, F.Cu at (88.8, 56.9)
- added J9: Conn_01x01_Male, Connector_PinHeader_2.54mm:PinHeader_1x01_P2.54mm_Vertical, F.Cu at (76.1, 23.3)
- added SW1: SWITCH-DIP10, Package_DIP:DIP-20_W7.62mm, F.Cu at (141.3, 61.4)
- C20: footprint Capacitor_SMD:C_0805_2012Metric -> Capacitor_THT:C_Rect_L7.0mm_W2.0mm_P5.00mm
- J7: moved to B.Cu
- JP1: footprint Connector_PinHeader_2.54mm:PinHeader_1x02_P2.54mm_Horizontal -> Connector_PinHeader_2.54mm:PinHeader_1x02_P2.54mm_Vertical
- moved C20 145.3 mm to (68.7, 97.3)
- moved Q10 142.8 mm to (75.2, 83.3), turned to 180 degrees
- moved R37 139.4 mm to (78.0, 97.0)
- moved R1 137.4 mm to (70.6, 105.5), turned to 180 degrees
- moved C2 134.5 mm to (83.3, 34.0), turned to 180 degrees
- moved R3 132.6 mm to (85.1, 100.7), turned to 270 degrees
- moved C12 129.1 mm to (71.9, 32.1), turned to 90 degrees
- moved C1 128.9 mm to (69.3, 32.2), turned to 90 degrees
- moved D3 124.2 mm to (93.3, 74.1)
- moved R29 123.3 mm to (96.2, 31.9), turned to 180 degrees
- moved U9 121.5 mm to (81.5, 76.5)
- moved R28 121.5 mm to (96.6, 103.0)
- moved R8 120.6 mm to (83.6, 58.7)
- moved C3 120.5 mm to (81.8, 67.6), turned to 270 degrees
- moved R33 119.9 mm to (83.6, 86.9)
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- renumbered D6 to LED1, D11 to LED2
Connections:
- net Net-(J4-Pad2) renamed /USB_N
- net Net-(J4-Pad3) renamed /USB_P
- J2 pad 1: (no net) -> Net-(J2-Pad1)
- J2 pad 6: (no net) -> Net-(J2-Pad6)
- J4 pad 4: (no net) -> Net-(J4-Pad4)
- J5 pad 1: (no net) -> Net-(J5-Pad1)
- J5 pad 4: (no net) -> Net-(J5-Pad4)
- J5 pad 6: (no net) -> Net-(J5-Pad6)
- J5 pad 7: (no net) -> Net-(J5-Pad7)
- J5 pad 8: (no net) -> Net-(J5-Pad8)
- J5 pad 9: (no net) -> Net-(J5-Pad9)
- J7 pad 1: (no net) -> Net-(J7-Pad1)
- J7 pad 11: (no net) -> Net-(J7-Pad11)
- J7 pad 12: (no net) -> Net-(J7-Pad12)
- J7 pad 13: (no net) -> Net-(J7-Pad13)
- J7 pad 15: (no net) -> Net-(J7-Pad15)
- J7 pad 16: (no net) -> Net-(J7-Pad16)
- J7 pad 17: (no net) -> Net-(J7-Pad17)
- J7 pad 18: (no net) -> Net-(J7-Pad18)
- J7 pad 22: (no net) -> Net-(J7-Pad22)
- J7 pad 24: (no net) -> Net-(J7-Pad24)
- J7 pad 26: (no net) -> Net-(J7-Pad26)
- J7 pad 28: (no net) -> Net-(J7-Pad28)
- J7 pad 32: (no net) -> Net-(J7-Pad32)
- J7 pad 33: (no net) -> Net-(J7-Pad33)
- J7 pad 35: (no net) -> Net-(J7-Pad35)
- J7 pad 36: (no net) -> Net-(J7-Pad36)
- J7 pad 37: (no net) -> Net-(J7-Pad37)
- J7 pad 38: (no net) -> Net-(J7-Pad38)
- J7 pad 40: (no net) -> Net-(J7-Pad40)
- J7 pad 7: (no net) -> Net-(J7-Pad7)
- R31 pad 1: Net-(R31-Pad1) -> /LED1
- R40 pad 1: Net-(R40-Pad1) -> /LED2
- R41 pad 1: Net-(R41-Pad1) -> /LED3
- R42 pad 1: Net-(R42-Pad1) -> /LED4
- R43 pad 1: Net-(R43-Pad1) -> /LED5
- R44 pad 1: Net-(R44-Pad1) -> /LED6
- U14 pad 10: /CURRENTSENSE -> /LINEVOLTAGE
- U14 pad 11: /LINEVOLTAGE -> /CURRENTSENSE
- U14 pad 12: /LINEVOLTAGE -> Net-(U14-Pad12)
- U14 pad 13: /TTX -> /REVERSE
- U14 pad 14: Net-(JP20-Pad1) -> /TTX
- U14 pad 17: Net-(JP16-Pad1) -> /KEYBOARD
- U14 pad 18: /REVERSE -> /TPON
- U14 pad 19: /KEYBOARD -> /VOLT1
- U14 pad 2: (no net) -> Net-(U14-Pad2)
- U14 pad 20: /TPON -> /VOLT0
- U14 pad 21: Net-(R43-Pad1) -> /CURR1
- U14 pad 22: Net-(R44-Pad1) -> /CURR0
- U14 pad 25: (no net) -> /HBAUD1
- U14 pad 26: (no net) -> /HBAUD0
- U14 pad 27: Net-(JP2-Pad2) -> /TPBAUD1
- U14 pad 28: Net-(JP3-Pad2) -> /TPBAUD0
- U14 pad 29: Net-(JP7-Pad1) -> /TEST1
- U14 pad 3: (no net) -> Net-(U14-Pad3)
- U14 pad 32: Net-(JP8-Pad1) -> /TEST0
- U14 pad 33: Net-(JP9-Pad1) -> /LED4
- U14 pad 38: Net-(JP10-Pad1) -> /LED5
- U14 pad 4: (no net) -> Net-(U14-Pad4)
- U14 pad 42: Net-(R31-Pad1) -> /LED6
- U14 pad 43: Net-(R40-Pad1) -> /LED1
- U14 pad 45: Net-(R41-Pad1) -> /LED2
- U14 pad 46: Net-(R42-Pad1) -> /LED3
- U3 pad 10: (no net) -> Net-(U3-Pad10)
- U3 pad 11: (no net) -> Net-(U3-Pad11)
- U3 pad 12: (no net) -> Net-(U3-Pad12)
- U3 pad 13: (no net) -> Net-(U3-Pad13)
- U3 pad 14: (no net) -> Net-(U3-Pad14)
- U3 pad 2: (no net) -> Net-(U3-Pad2)
- U3 pad 22: (no net) -> Net-(U3-Pad22)
- U3 pad 23: (no net) -> Net-(U3-Pad23)
- U3 pad 27: (no net) -> Net-(U3-Pad27)
- U3 pad 28: (no net) -> Net-(U3-Pad28)
- U3 pad 3: (no net) -> Net-(U3-Pad3)
- U3 pad 6: (no net) -> Net-(U3-Pad6)
- U3 pad 9: (no net) -> Net-(U3-Pad9)
- U4 pad 11: (no net) -> Net-(U4-Pad11)
- U4 pad 14: (no net) -> Net-(U4-Pad14)
- U4 pad 8: (no net) -> Net-(U4-Pad8)
- U4 pad 9: (no net) -> Net-(U4-Pad9)
Routing:
- net GND: track 0.00 -> 531.0 mm, vias 0 -> 28
- net +3V3: track 0.00 -> 247.4 mm, vias 0 -> 18
- net /TX: track 0.00 -> 136.2 mm, vias 0 -> 9
- net +5V: track 0.00 -> 111.6 mm, vias 0 -> 6
- net Net-(JP11-Pad1): track 0.00 -> 108.7 mm, vias 0 -> 5
- net /KEYBOARD: track 0.00 -> 98.6 mm, vias 0 -> 2
- net /TPON: track 0.00 -> 78.6 mm, vias 0 -> 4
- net Net-(J11-Pad1): track 0.00 -> 57.7 mm, vias 0 -> 5
- net Net-(C4-Pad1): track 0.00 -> 53.0 mm, vias 0 -> 1
- net /CURRENTSENSE: track 0.00 -> 49.3 mm, vias 0 -> 2
- net Net-(D4-Pad1): track 0.00 -> 48.9 mm
- net /REVERSE: track 0.00 -> 48.7 mm
- net /TTX: track 0.00 -> 47.0 mm, vias 0 -> 4
- net Net-(R7-Pad1): track 0.00 -> 44.3 mm, vias 0 -> 2
- net Net-(C14-Pad1): track 0.00 -> 42.4 mm, vias 0 -> 2
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- added copper zone on B.Cu, net +3V3
- added copper zone on B.Cu, net +5V
- added copper zone on F.Cu, net GND
Other:
- board outline added: 83.5 x 97.5 mm
- board text added: "+5V CENTER PIN POSITIVE"
- board text added: "BOOT"
- board text added: "CLRX"
- board text added: "CONF0"
- board text added: "CONF1"
- board text added: "CONF2"
- board text added: "CURRENT LOOP"
- board text added: "GND"
- board text added: "HV"
- board text added: "Mattis Lind 2022"
- board text added: "RASPIRX"
- board text added: "RESET"
- board text added: "RS-232"
- board text added: "RS232RX"
- board text added: "RX"
- board text added: "SENSE"
- board text added: "TELEPRINTER"
- board text added: "TX"
- board text added: "USBRX"
- board text added: "WP"
- board text added: "https://github.com/MattisLind/teleprinterHat"
- board text added: "www.datormuseum.se"

Commit message: Added pdf and SVG
Connections:
- net Net-(J6-Pad2) renamed /SWDIO
- net Net-(J6-Pad3) renamed /SWCLK
- U14 pad 12: Net-(U14-Pad12) -> /LINECURRENT
- U14 pad 39: /MISO -> /SCK
- U14 pad 40: /MOSI -> /MISO
- U14 pad 41: /SCK -> /MOSI
Routing:
- net /LINECURRENT: track 2.17 -> 31.7 mm, vias 0 -> 2
- net /MISO: track 37.5 -> 36.3 mm
- net /CURRENTSENSE: track 49.3 -> 48.4 mm
- net /SCK: track 35.1 -> 35.5 mm, vias 4 -> 2
- net /MOSI: track 38.5 -> 38.6 mm, vias 2 -> 4
