File: hardware/TeleprinterHat/TeleprinterHat.sch (KiCad schematic (older format))
At the start: 144 parts, among them J1 LOOP/SELECTOR, J2 KEYBOARD, J3 SSR, J4 USB_B_Micro, J5 RS232, J6 JTAG, J7 RasPi GPIO, J8 AudioJack4, K1 FINDER-30.22, Q1 STD25NF20, Q10 FMMT625, Q2 MMBT3904, Q3 FMMT625, Q4 FMMT625, Q5 MMBT5551L, Q6 MMBT5551L, Q7 MMBTA42L, Q8 SQ2325ES, Q9 FMMT597, U1 NCP1117-3.3_TO252, U10 TLV3502, U11 MCP6004, U12 MCP6004, U13 74LVC1G04, U14 STM32F103C8Tx, U2 74LVC1G04, U3 FT232RL, U4 MAX3232, U5 MC34063, U6 24LC32, U7 SFH690BT, U8 SFH690BT, U9 IR44273, Y1 8MHz

Commit message: Ready for routing board.
Parts:
- removed J1: LOOP/SELECTOR, symbol Connector:AudioJack2
- removed J2: KEYBOARD, symbol Connector:AudioJack2
- removed J3: SSR, symbol Connector:AudioJack2
- removed J8: AudioJack4, symbol Connector:AudioJack4
- removed K1: FINDER-30.22, Relay_THT:Relay_DPDT_Finder_30.22, symbol Relay:FINDER-30.22
- removed U6: 24LC32, symbol Memory_EEPROM:24LC32
- added J1, J2: RJ12, Connector_RJ:RJ12_Amphenol_54601, symbol Connector:RJ12
- added K1: EA2-5NU, Package_DIP:DIP-10_W7.62mm, symbol EA2-5NU:EA2-5NU
- added U6: 24LC32AT-IOT, Package_TO_SOT_SMD:SOT-23-5_HandSoldering, symbol 24LC32AT-SOT-23-5:24LC32AT-IOT
- C1, C10, C11, C12, C13, C14, C15, C16, C17, C18, C19, C2, C20, C21, C22, C23, C24, C25, C3, C6, C7, C8, C9: footprint (none) -> Capacitor_SMD:C_0805_2012Metric
- C4: footprint (none) -> Capacitor_SMD:CP_Elec_10x7.7
- C5: footprint (none) -> Capacitor_THT:CP_Radial_D8.0mm_P3.50mm
- D1, D10, D9: footprint (none) -> Diode_SMD:D_SOD-123
- D11, D6: footprint (none) -> LED_SMD:LED_Avago_PLCC6_3x2.8mm
- D12, D3, D4, Q10, Q3, Q4, Q7, Q8, Q9: footprint (none) -> Package_TO_SOT_SMD:SOT-23
- D2, D5: footprint (none) -> Diode_SMD:D_SMB_Handsoldering
- D7, D8: footprint (none) -> LED_SMD:LED_0805_2012Metric_Castellated
- F1: footprint (none) -> Fuse:Fuse_0603_1608Metric_Pad1.05x0.95mm_HandSolder
- J4: footprint (none) -> Connector_USB:USB_Micro-B_Amphenol_10103594-0001LF_Horizontal
- J5: footprint (none) -> Connector_Dsub:DSUB-9_Female_Horizontal_P2.77x2.84mm_EdgePinOffset9.90mm_Housed_MountingHolesOffset11.32mm
- J6: footprint (none) -> Connector_PinHeader_2.54mm:PinHeader_1x04_P2.54mm_Vertical
- J7: footprint (none) -> Connector_PinSocket_2.54mm:PinSocket_2x20_P2.54mm_Vertical
- JP1: footprint (none) -> Connector_PinHeader_2.54mm:PinHeader_1x02_P2.54mm_Horizontal
- JP10, JP11, JP12, JP13, JP14, JP15, JP16, JP17, JP18, JP2, JP20, JP21, JP3, JP4, JP5, JP6, JP7, JP8, JP9: footprint (none) -> Connector_PinHeader_2.54mm:PinHeader_1x02_P2.54mm_Vertical
- JP19: value RESET -> BOOT; footprint (none) -> Connector_PinHeader_2.54mm:PinHeader_1x02_P2.54mm_Vertical
- L1: footprint (none) -> General:Wurth TIF Radial 1018
- L2: footprint (none) -> Inductor_THT:L_Radial_D7.0mm_P3.00mm
- L4: footprint (none) -> Inductor_THT:L_Radial_D12.0mm_P6.00mm_MuRATA_1900R
- Q1: footprint (none) -> Package_TO_SOT_SMD:TO-252-3_TabPin2
- R1, R10, R11, R12, R13, R14, R15, R16, R17, R18, R19, R2, R20, R21, R22, R23, R24, R25, R26, R27, R28, R29, R3, R30, R31, R32, R33, R34, R35, R36, R37, R38, R39, R4, R40, R41, R42, R43, R44, R45, R46, R47, R48, R5, R6, R7, R8, R9: footprint (none) -> Resistor_SMD:R_0805_2012Metric
- U10: footprint (none) -> Package_TO_SOT_SMD:SOT-23-8_Handsoldering
- U11: footprint (none) -> Package_SO:SOIC-14_3.9x8.7mm_P1.27mm
- U11: renamed from U12; footprint (none) -> Package_SO:SOIC-14_3.9x8.7mm_P1.27mm
- U13, U2, U9: footprint (none) -> Package_TO_SOT_SMD:SOT-23-5_HandSoldering
- U4: footprint (none) -> Package_SO:SOIC-16_3.9x9.9mm_P1.27mm
- U5: footprint (none) -> Package_SO:SOIC-8_3.9x4.9mm_P1.27mm
- Y1: footprint (none) -> Crystal:Crystal_SMD_HC49-SD
Connections:
- net labels added: PRINTER+, PRINTER-
- wire segments 561 -> 560
- no-connect marks 47 -> 51
Other:
- note added: "649-54601-906001WPLF"
- note removed: "Mouser: 490-MJ-2506N"
- note removed: "Mouser: 490-SJ1-42514"
- moved on the sheet: R1

Commit message: Almost ready!
Parts:
- removed JP10: CURR1, Connector_PinHeader_2.54mm:PinHeader_1x02_P2.54mm_Vertical, symbol Device:Jumper_NC_Small
- removed JP15: TPBAUD0, Connector_PinHeader_2.54mm:PinHeader_1x02_P2.54mm_Vertical, symbol Device:Jumper_NC_Small
- removed JP16: TPBAUD1, Connector_PinHeader_2.54mm:PinHeader_1x02_P2.54mm_Vertical, symbol Device:Jumper_NC_Small
- removed JP2: VOLT0, Connector_PinHeader_2.54mm:PinHeader_1x02_P2.54mm_Vertical, symbol Device:Jumper_NC_Small
- removed JP20: TEST1, Connector_PinHeader_2.54mm:PinHeader_1x02_P2.54mm_Vertical, symbol Device:Jumper_NC_Small
- removed JP21: TEST2, Connector_PinHeader_2.54mm:PinHeader_1x02_P2.54mm_Vertical, symbol Device:Jumper_NC_Small
- removed JP3: VOLT1, Connector_PinHeader_2.54mm:PinHeader_1x02_P2.54mm_Vertical, symbol Device:Jumper_NC_Small
- removed JP7: HBAUD0, Connector_PinHeader_2.54mm:PinHeader_1x02_P2.54mm_Vertical, symbol Device:Jumper_NC_Small
- removed JP8: HBAUD1, Connector_PinHeader_2.54mm:PinHeader_1x02_P2.54mm_Vertical, symbol Device:Jumper_NC_Small
- removed JP9: CURR0, Connector_PinHeader_2.54mm:PinHeader_1x02_P2.54mm_Vertical, symbol Device:Jumper_NC_Small
- added H1, H2, H3, H4, H5, H6, H7, H8: MountingHole, MountingHole:MountingHole_2.7mm_M2.5, symbol Mechanical:MountingHole
- added J10, J11, J8, J9: Conn_01x01_Male, Connector_PinHeader_2.54mm:PinHeader_1x01_P2.54mm_Vertical, symbol Connector:Conn_01x01_Male
- added J3: DC_JACK, Connector_BarrelJack:BarrelJack_Wuerth_6941xx301002, symbol tinkerforge:DC_JACK
- added SW1: SWITCH-DIP10, Package_DIP:DIP-20_W7.62mm, symbol tinkerforge:SWITCH-DIP10
- C1, C10, C11, C13, C14, C15, C16, C17, C18, C19, C2, C21, C22, C23, C24, C25, C3, C6, C7, C8, C9: symbol Device:C_Small -> TeleprinterHat-rescue:C_Small-Device
- C12, C4, C5: symbol Device:CP_Small -> TeleprinterHat-rescue:CP_Small-Device
- C20: footprint Capacitor_SMD:C_0805_2012Metric -> Capacitor_THT:C_Rect_L7.0mm_W2.0mm_P5.00mm; symbol Device:C_Small -> TeleprinterHat-rescue:C_Small-Device
- D1: symbol Device:D_Zener_Small -> TeleprinterHat-rescue:D_Zener_Small-Device
- D10, D12, D2, D3, D4, D9: symbol Device:D_Small -> TeleprinterHat-rescue:D_Small-Device
- D11, D6: symbol Device:LED_RGB -> TeleprinterHat-rescue:LED_RGB-Device
- D5: symbol tinkerforge:TVS -> TeleprinterHat-rescue:TVS-tinkerforge
- D7, D8: symbol Device:LED -> TeleprinterHat-rescue:LED-Device
- F1: symbol Device:Fuse_Small -> TeleprinterHat-rescue:Fuse_Small-Device
- J7: symbol Connector_Generic:Conn_02x20_Odd_Even -> TeleprinterHat-rescue:Conn_02x20_Odd_Even-Connector_Generic
- JP1: footprint Connector_PinHeader_2.54mm:PinHeader_1x02_P2.54mm_Horizontal -> Connector_PinHeader_2.54mm:PinHeader_1x02_P2.54mm_Vertical; symbol Device:Jumper_NC_Small -> TeleprinterHat-rescue:Jumper_NC_Small-Device
- JP11, JP12, JP13, JP14, JP17, JP18, JP19, JP4, JP5, JP6: symbol Device:Jumper_NC_Small -> TeleprinterHat-rescue:Jumper_NC_Small-Device
- K1: symbol EA2-5NU:EA2-5NU -> TeleprinterHat-rescue:EA2-5NU-EA2-5NU
- L1, L2: symbol Device:L -> TeleprinterHat-rescue:L-Device
- L4: symbol Device:L_Core_Ferrite_Small -> TeleprinterHat-rescue:L_Core_Ferrite_Small-Device
- Q1: symbol Device:Q_NMOS_GDS -> TeleprinterHat-rescue:Q_NMOS_GDS-Device
- Q10, Q3, Q4, Q7: symbol Device:Q_NPN_BEC -> TeleprinterHat-rescue:Q_NPN_BEC-Device
- Q2: symbol Transistor_BJT:MMBT3904 -> TeleprinterHat-rescue:MMBT3904-Transistor_BJT
- Q5, Q6: symbol Transistor_BJT:MMBT5551L -> TeleprinterHat-rescue:MMBT5551L-Transistor_BJT
- Q8: symbol Device:Q_PMOS_GDS -> TeleprinterHat-rescue:Q_PMOS_GDS-Device
- Q9: symbol Device:Q_PNP_BEC -> TeleprinterHat-rescue:Q_PNP_BEC-Device
- R1, R19, R20, R3, R31, R40, R41, R42, R43, R44: symbol Device:R -> TeleprinterHat-rescue:R-Device
- R10, R11, R12, R13, R14, R15, R16, R17, R18, R2, R21, R22, R23, R24, R25, R26, R27, R28, R29, R30, R32, R33, R34, R35, R36, R37, R38, R39, R4, R45, R46, R47, R48, R5, R6, R7, R8, R9: symbol Device:R_Small -> TeleprinterHat-rescue:R_Small-Device
- U1: symbol Regulator_Linear:NCP1117-3.3_TO252 -> TeleprinterHat-rescue:NCP1117-3.3_TO252-Regulator_Linear
- U10: symbol tlv3502:TLV3502 -> TeleprinterHat-rescue:TLV3502-tlv3502
- U11: symbol Amplifier_Operational:MCP6004 -> TeleprinterHat-rescue:MCP6004-Amplifier_Operational
- U13, U2: symbol 74xGxx:74LVC1G04 -> TeleprinterHat-rescue:74LVC1G04-74xGxx
- U14: symbol MCU_ST_STM32F1:STM32F103C8Tx -> TeleprinterHat-rescue:STM32F103C8Tx-MCU_ST_STM32F1
- U3: symbol Interface_USB:FT232RL -> TeleprinterHat-rescue:FT232RL-Interface_USB
- U4: symbol Interface_UART:MAX232 -> TeleprinterHat-rescue:MAX232-Interface_UART
- U5: symbol MC34063:MC34063 -> TeleprinterHat-rescue:MC34063-MC34063
- U6: symbol 24LC32AT-SOT-23-5:24LC32AT-IOT -> TeleprinterHat-rescue:24LC32AT-IOT-24LC32AT-SOT-23-5
- U7, U8: symbol Isolator:LTV-355T -> TeleprinterHat-rescue:LTV-355T-Isolator
- U9: symbol irs44273:IRS44273 -> TeleprinterHat-rescue:IRS44273-irs44273
- Y1: symbol Device:Crystal_Small -> TeleprinterHat-rescue:Crystal_Small-Device
Connections:
- net labels added: CURR0, CURR1, HBAUD0, HBAUD1, LED1, LED2, LED3, LED4, LED5, LED6, TEST0, TEST1, TPBAUD0, TPBAUD1, USB_N, USB_P, VOLT0, VOLT1
- wire segments 560 -> 573
- no-connect marks 51 -> 52

Commit message: Added pdf and SVG
Parts:
- D7: value RX -> RX GREEN
- D8: value TX -> TX RED
- R19: value 470 -> 1,2k
- R20: value 470 -> 1,5k
- R31, R42: value 470 -> 2k
- R40, R43: value 470 -> 2,7k
- R41, R44: value 470 -> 3,3k
- renumbered D6 to LED1, D11 to LED2
Connections:
- net labels added: SWCLK, SWDIO
- wire segments 573 -> 577
- no-connect marks 52 -> 51
Other:
- moved on the sheet: D7, D8
Changed lines of the file:
@@
 P 11900 8150
 F 0 "D8" V 12000 8250 50  0000 R CNN
-F 1 "TX" V 11800 8250 50  0000 R CNN
+F 1 "TX RED" H 12050 8300 50  0000 R CNN
 F 2 "LED_SMD:LED_0805_2012Metric_Castellated" H 11900 8150 50  0001 C CNN
 F 3 "~" H 11900 8150 50  0001 C CNN
 	1    11900 8150
-	0    -1   -1   0
+	0    1    1    0
 $EndComp
 $Comp
@@
 P 11650 8150
 F 0 "D7" V 11750 8150 50  0000 R CNN
-F 1 "RX" V 11550 8250 50  0000 R CNN
+F 1 "RX GREEN" H 11700 8000 50  0000 R CNN
 F 2 "LED_SMD:LED_0805_2012Metric_Castellated" H 11650 8150 50  0001 C CNN
 F 3 "~" H 11650 8150 50  0001 C CNN
 	1    11650 8150
-	0    -1   -1   0
+	0    1    1    0
 $EndComp
 $Comp
@@
 	1    0    0    -1
 $EndComp
-Wire Wire Line
-	11150 8750 11150 7850
 $Comp
 L TeleprinterHat-rescue:GND-power #PWR0124
@@
 P 11650 7800
 F 0 "R19" H 11580 7754 50  0000 R CNN
-F 1 "470" H 11580 7845 50  0000 R CNN
+F 1 "1,2k" H 11580 7845 50  0000 R CNN
 F 2 "Resistor_SMD:R_0805_2012Metric" V 11580 7800 50  0001 C CNN
 F 3 "~" H 11650 7800 50  0001 C CNN
@@
 P 11900 7800
 F 0 "R20" H 11830 7754 50  0000 R CNN
-F 1 "470" H 11830 7845 50  0000 R CNN
+F 1 "1,5k" H 11830 7845 50  0000 R CNN
 F 2 "Resistor_SMD:R_0805_2012Metric" V 11830 7800 50  0001 C CNN
 F 3 "~" H 11900 7800 50  0001 C CNN
@@
 	11900 7650 11900 7450
 Connection ~ 11900 7450
-$Comp
-L TeleprinterHat-rescue:GND-power #PWR0127
-U 1 1 684F8309
-P 11650 8350
-F 0 "#PWR0127" H 11650 8100 50  0001 C CNN
-F 1 "GND" H 11655 8177 50  0000 C CNN
-F 2 "" H 11650 8350 50  0001 C CNN
-F 3 "" H 11650 8350 50  0001 C CNN
-	1    11650 8350
-	1    0    0    -1
-$EndComp
-Wire Wire Line
-	11650 8350 11650 8300
-Wire Wire Line
-	11650 8300 11900 8300
-Connection ~ 11650 8300
 Wire Wire Line
 	10700 7550 11650 7550
@@
 	8900 5150 8900 5100
 Wire Wire Line
-	11150 7850 10700 7850
+	11050 7850 10700 7850
 Wire Wire Line
-	11050 8750 11050 7950
-Wire Wire Line
-	11050 7950 10700 7950
+	11150 7950 10700 7950
 Wire Wire Line
 	11200 8050 10700 8050
@@
 P 7850 8350
 F 0 "R44" V 7950 8450 50  0000 C CNN
-F 1 "470" V 7950 8250 50  0000 C CNN
+F 1 "3,3k" V 7950 8250 50  0000 C CNN
 F 2 "Resistor_SMD:R_0805_2012Metric" V 7780 8350 50  0001 C CNN
 F 3 "~" H 7850 8350 50  0001 C CNN
@@
 P 7850 8150
 F 0 "R43" V 7950 8250 50  0000 C CNN
-F 1 "470" V 7950 8050 50  0000 C CNN
+F 1 "2,7k" V 7950 8050 50  0000 C CNN
 F 2 "Resistor_SMD:R_0805_2012Metric" V 7780 8150 50  0001 C CNN
 F 3 "~" H 7850 8150 50  0001 C CNN
@@
 P 7850 7950
 F 0 "R42" V 7950 8050 50  0000 C CNN
-F 1 "470" V 7950 7850 50  0000 C CNN
+F 1 "2k" V 7950 7850 50  0000 C CNN
 F 2 "Resistor_SMD:R_0805_2012Metric" V 7780 7950 50  0001 C CNN
 F 3 "~" H 7850 7950 50  0001 C CNN
@@
 P 7850 7500
 F 0 "R41" V 7950 7600 50  0000 C CNN
-F 1 "470" V 7950 7400 50  0000 C CNN
+F 1 "3,3k" V 7950 7400 50  0000 C CNN
 F 2 "Resistor_SMD:R_0805_2012Metric" V 7780 7500 50  0001 C CNN
 F 3 "~" H 7850 7500 50  0001 C CNN
@@
 P 7850 7300
 F 0 "R40" V 7950 7400 50  0000 C CNN
-F 1 "470" V 7950 7200 50  0000 C CNN
+F 1 "2,7k" V 7950 7200 50  0000 C CNN
 F 2 "Resistor_SMD:R_0805_2012Metric" V 7780 7300 50  0001 C CNN
 F 3 "~" H 7850 7300 50  0001 C CNN
@@
 P 7850 7100
 F 0 "R31" V 7950 7200 50  0000 C CNN
-F 1 "470" V 7950 7000 50  0000 C CNN
+F 1 "2k" V 7950 7000 50  0000 C CNN
 F 2 "Resistor_SMD:R_0805_2012Metric" V 7780 7100 50  0001 C CNN
 F 3 "~" H 7850 7100 50  0001 C CNN
@@
 Text Label 9000 6550 0    50   ~ 0
 TPON
-Text Label 9000 6850 0    50   ~ 0
-MISO
 Text Label 9000 6950 0    50   ~ 0
-MOSI
+MISO
 Text Label 9000 7050 0    50   ~ 0
+MOSI
+Text Label 9000 6850 0    50   ~ 0
 SCK
 $Comp
@@
 Mouser:80-EDK107M016A9GAA\n100uF 16V
 $Comp
-L TeleprinterHat-rescue:LED_RGB-Device D6
+L TeleprinterHat-rescue:LED_RGB-Device LED1
 U 1 1 61147F80
 P 7350 7300
-F 0 "D6" H 7350 7797 50  0000 C CNN
+F 0 "LED1" H 7350 7797 50  0000 C CNN
 F 1 "LED_RGB" H 7350 7706 50  0000 C CNN
 F 2 "LED_SMD:LED_Avago_PLCC6_3x2.8mm" H 7350 7250 50  0001 C CNN
@@
 $EndComp
 $Comp
-L TeleprinterHat-rescue:LED_RGB-Device D11
+L TeleprinterHat-rescue:LED_RGB-Device LED2
 U 1 1 611483D9
 P 7350 8150
-F 0 "D11" H 7350 8647 50  0000 C CNN
+F 0 "LED2" H 7350 8647 50  0000 C CNN
 F 1 "LED_RGB" H 7350 8556 50  0000 C CNN
 F 2 "LED_SMD:LED_Avago_PLCC6_3x2.8mm" H 7350 8100 50  0001 C CNN
@@
 Text Label 10850 7350 0    50   ~ 0
 TEST1
-NoConn ~ 10700 6750
 $Comp
 L power:GND #PWR03
@@
 Text Label 1950 8600 0    50   ~ 0
 USB_N
+Text Label 10750 7950 0    50   ~ 0
+SWCLK
+Text Label 10800 7850 0    50   ~ 0
+SWDIO
+Wire Wire Line
+	10700 6750 11150 6750
+Text Label 10750 6750 0    50   ~ 0
+LINECURRENT
+Wire Wire Line
+	11650 8300 11650 8450
+Wire Wire Line
+	11650 8450 11900 8450
+Wire Wire Line
+	11900 8450 11900 8300
+$Comp
+L TeleprinterHat-rescue:+3V3-power #PWR?
+U 1 1 623071EA
+P 11350 8350
+F 0 "#PWR?" H 11350 8200 50  0001 C CNN
+F 1 "+3V3" H 11365 8523 50  0000 C CNN
+F 2 "" H 11350 8350 50  0001 C CNN
+F 3 "" H 11350 8350 50  0001 C CNN
+	1    11350 8350
+	1    0    0    -1
+$EndComp
+Wire Wire Line
+	11350 8350 11350 8450
+Wire Wire Line
+	11350 8450 11650 8450
+Connection ~ 11650 8450
+Wire Wire Line
+	11150 8750 11150 7950
+Wire Wire Line
+	11050 8750 11050 7850
 $EndSCHEMATC
